File: hardware/board-files/nightLight-r2/nightLight.kicad_sch (KiCad schematic)
At the start: 25 parts, among them IC1 PAM2401SCADJ, J1 Conn_01x03, J2 Conn_01x03, J3 Conn_01x03, J4 Conn_01x03, SW2 TILT, U1 USB-C_PWR, U2 ATtiny1614-SS, U3 MCP73831-2-OT

Commit message: Finished schematic, started PCB. Figuring out copper zones
Parts:
- removed C2: 22uF, Capacitor_SMD:C_1206_3216Metric, symbol Device:C
- removed J4: Conn_01x03, Connector_PinHeader_2.54mm:PinHeader_1x03_P2.54mm_Vertical_SMD_Pin1Left, symbol Connector_Generic:Conn_01x03
- removed U1: USB-C_PWR, myFootprintDesigns:USB-C_PWR, symbol myDesigns:USB-C_PWR
- added C5, C6: 22uF, Capacitor_SMD:C_1206_3216Metric, symbol Device:C
- added C7: 0.1uF, Capacitor_SMD:C_1206_3216Metric, symbol Device:C
- added J1: USB_C_Receptacle_PowerOnly_6P, myFootprintDesigns:USB-C_PWR, symbol Connector:USB_C_Receptacle_PowerOnly_6P
- added J5: Conn_01x03, Connector_PinHeader_2.54mm:PinHeader_1x03_P2.54mm_Vertical_SMD_Pin1Left, symbol Connector_Generic:Conn_01x03
- added J6: Conn_01x05_Pin, Connector_PinSocket_2.54mm:PinSocket_1x05_P2.54mm_Vertical_SMD_Pin1Left, symbol Connector:Conn_01x05_Pin
- added R1: 0, Resistor_SMD:R_1206_3216Metric, symbol Device:R_US
- added R10, R9: 100k, Resistor_SMD:R_1206_3216Metric, symbol Device:R_US
- added R11: 10k, Resistor_SMD:R_1206_3216Metric, symbol Device:R_US
- added R2, R4: 5.1k, Resistor_SMD:R_1206_3216Metric, symbol Device:R_US
- added S1: PTS526_SM08_SMTR2_LFS, PTS526_SM08_SMTR2_LFS:SW_PTS526_SM08_SMTR2_LFS, symbol PTS526_SM08_SMTR2_LFS:PTS526_SM08_SMTR2_LFS
- R13: renamed from R1; value 10k -> 1M
- renumbered C5 to C2, J1 to J2, J2 to J3, J3 to J4, R2 to R12, R6 to R5, R7 to R6, R4 to R7, R5 to R8, SW2 to SW1, U3 to U1
Connections:
- net +5V: now also C5.1, C6.1, C7.1, J6.5 (Pin_5), R11.1
- net GND: now also C5.2, C6.2, C7.2, J1.A12 (GND), J1.B12 (GND), J6.1 (Pin_1), R10.2, R2.2, R4.2, S1.1, S1.2
- net VBATT: now also R1.2, R9.1; no longer C1.1, IC1.3 (VIN), L1.1, R3.1
- net Batt_M: now reaches U2.2 (PA4)
- net Batt_M: now also R10.1, R9.2; no longer J2.2 (Pin_2)
- net UPDI: now reaches U2.10 (~{RESET}/PA0)
- net UPDI: now also J6.4 (Pin_4)
- net PA_1: now reaches U2.11 (PA1)
- net PA_1: now also J5.1 (Pin_1)
- net PA_2: now reaches U2.12 (PA2)
- net PA_2: now also J5.2 (Pin_2)
- net PA_3: now reaches U2.13 (PA3)
- net PA_3: now also J5.3 (Pin_3)
- net Send: now reaches R13.1, U2.3 (PA5)
- net Return: now reaches B1.1, R13.2, U2.4 (PA6)
- net Tilt_SW: now reaches R12.2, SW1.1, U2.5 (PA7)
- net RX: now reaches U2.6 (PB3)
- net RX: now also J6.3 (Pin_3)
- net TX: now reaches U2.7 (PB2)
- net TX: now also J6.2 (Pin_2)
- net LED_DATA: now reaches U2.8 (PB1)
- net LED_DATA: now also J2.2 (Pin_2)
- net RST_SW: now reaches U2.9 (PB0)
- net RST_SW: now also R11.2, S1.3, S1.4
- net at C2.1, R6.1, U1.4 (V_{DD}): now also J1.A9 (VBUS), J1.B9 (VBUS)
- new net: C1.1, IC1.3 (VIN), L1.1, R1.1, R3.1
- new net: J1.B5 (CC2), R2.1
- new net: J1.A5 (CC1), R4.1
- no-connect marks 8 -> 2
Other:
- note added: "LED String"
- note added: "Programming"
- note added: "Spare"
- company: (none) -> Cameron Gillingham
- title: (none) -> Night Light
- moved on the sheet: B1, C2, J2, J3, J4, R12, R13, SW1, U2

Commit message: Finished first PCB revision
Parts:
- removed D1: IN-S124ARUW, IN-S124ARUW:LED_IN-S124ARUW, symbol IN-S124ARUW:IN-S124ARUW
- added LED1: IN-S124ARUW, INS124ARUW, symbol newIN-S124ARUW:IN-S124ARUW
Connections:
- net VBATT: no longer R9.1
- net vBATT: now reaches C1.1, IC1.3 (VIN), L1.1, R1.1, R3.1
- net vBATT: now also R9.1
- net at R6.2: now also LED1.2 (A)
- net at U1.1 (STAT): now also LED1.1 (K)
Changed lines of the file:
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@@
+    (stroke (width 0) (type default))
+  )
+  (wire (pts (xy 109.22 43.18) (xy 109.22 45.72))
     (stroke (width 0) (type default))
   )
@@
   )
   (wire (pts (xy 74.93 77.47) (xy 74.93 76.2))
-    (stroke (width 0) (type default))
-  )
-  (wire (pts (xy 109.22 43.18) (xy 109.22 48.26))
     (stroke (width 0) (type default))
   )
@@
     (effects (font (size 2 2) (color 237 0 0 1)) (justify left bottom))
   )
-  (global_label "VBATT" (shape input) (at 194.31 124.46 90) (fields_autoplaced)
+  (global_label "vBATT" (shape input) (at 194.31 124.46 90) (fields_autoplaced)
     (effects (font (size 1.27 1.27)) (justify left))
-    (property "Intersheetrefs" "${INTERSHEET_REFS}" (at 194.31 116.0924 90)
+    (property "Intersheetrefs" "${INTERSHEET_REFS}" (at 194.31 116.2134 90)
       (effects (font (size 1.27 1.27)) (justify left) hide)
     )
@@
     )
   )
+  (global_label "vBATT" (shape input) (at 41.91 130.81 180) (fields_autoplaced)
+    (effects (font (size 1.27 1.27)) (justify right))
+    (property "Intersheetrefs" "${INTERSHEET_REFS}" (at 33.6634 130.81 0)
+      (effects (font (size 1.27 1.27)) (justify right) hide)
+    )
+  )
   (global_label "RST_SW" (shape input) (at 214.63 131.445 180) (fields_autoplaced)
     (effects (font (size 1.27 1.27)) (justify right))
@@
     )
   )
-  (netclass_flag "" (length 1) (shape dot) (at 109.22 46.99 270) (fields_autoplaced)
+  (netclass_flag "" (length 1) (shape dot) (at 109.22 44.45 270) (fields_autoplaced)
     (effects (font (size 1.27 1.27)) (justify right bottom))
-    (property "Netclass" "power" (at 110.22 46.2915 90)
+    (property "Netclass" "signal" (at 110.22 43.7515 90)
       (effects (font (size 1.27 1.27) italic) (justify left) hide)
     )
@@
   (netclass_flag "" (length 1) (shape dot) (at 102.87 68.58 180) (fields_autoplaced)
     (effects (font (size 1.27 1.27)) (justify right bottom))
-    (property "Netclass" "power" (at 103.5685 69.58 0)
+    (property "Netclass" "signal" (at 103.5685 69.58 0)
       (effects (font (size 1.27 1.27) italic) (justify left) hide)
     )
@@
     )
   )
+  (symbol (lib_id "newIN-S124ARUW:IN-S124ARUW") (at 109.22 60.96 90) (unit 1)
+    (in_bom yes) (on_board yes) (dnp no) (fields_autoplaced)
+    (property "Reference" "LED1" (at 113.03 52.07 90)
+      (effects (font (size 1.27 1.27)) (justify right))
+    )
+    (property "Value" "IN-S124ARUW" (at 113.03 54.61 90)
+      (effects (font (size 1.27 1.27)) (justify right))
+    )
+    (property "Footprint" "INS124ARUW" (at 202.87 48.26 0)
+      (effects (font (size 1.27 1.27)) (justify left bottom) hide)
+    )
+    (property "Datasheet" "http://www.inolux-corp.com/datasheet/SMDLED/Mono%20Color%20Reverse%20Mount/IN-S124AR%20Series_V1.0.pdf" (at 302.87 48.26 0)
+      (effects (font (size 1.27 1.27)) (justify left bottom) hide)
+    )
+    (property "Height" "1.1" (at 502.87 48.26 0)
+      (effects (font (size 1.27 1.27)) (justify left bottom) hide)
+    )
+    (property "Mouser Part Number" "743-IN-S124ARUW" (at 602.87 48.26 0)
+      (effects (font (size 1.27 1.27)) (justify left bottom) hide)
+    )
+    (property "Mouser Price/Stock" "https://www.mouser.co.uk/ProductDetail/Inolux/IN-S124ARUW?qs=qSfuJ%252Bfl%2Fd749ba9g3nPiA%3D%3D" (at 702.87 48.26 0)
+      (effects (font (size 1.27 1.27)) (justify left bottom) hide)
+    )
+    (property "Manufacturer_Name" "Inolux" (at 802.87 48.26 0)
+      (effects (font (size 1.27 1.27)) (justify left bottom) hide)
+    )
+    (property "Manufacturer_Part_Number" "IN-S124ARUW" (at 902.87 48.26 0)
+      (effects (font (size 1.27 1.27)) (justify left bottom) hide)
+    )
+    (pin "2")
+    (pin "1")
+    (instances
+      (project "nightLight"
+        (path "/203033dd-6a13-4262-9a98-8b29445e90e8"
+          (reference "LED1") (unit 1)
+        )
+      )
+    )
+  )
   (symbol (lib_id "power:GND") (at 115.57 77.47 0) (unit 1)
     (in_bom yes) (on_board yes) (dnp no) (fields_autoplaced)
@@
         )
       )
-    )
-  )
-  (symbol (lib_id "IN-S124ARUW:IN-S124ARUW") (at 109.22 55.88 270) (unit 1)
-    (in_bom yes) (on_board yes) (dnp no) (fields_autoplaced)
-    (property "Reference" "D1" (at 114.3 52.6034 90)
-      (effects (font (size 1.27 1.27)) (justify left))
-    )
-    (property "Value" "IN-S124ARUW" (at 114.3 55.1434 90)
-      (effects (font (size 1.27 1.27)) (justify left) hide)
-    )
-    (property "Footprint" "IN-S124ARUW:LED_IN-S124ARUW" (at 109.22 55.88 0)
-      (effects (font (size 1.27 1.27)) (justify bottom) hide)
-    )
-    (property "Datasheet" "" (at 109.22 55.88 0)
-      (effects (font (size 1.27 1.27)) hide)
-    )
-    (property "MF" "Inolux" (at 109.22 55.88 0)
-      (effects (font (size 1.27 1.27)) (justify bottom) hide)
-    )
-    (property "MOUSER-PURCHASE-URL" "https://snapeda.com/shop?store=Mouser&id=2130298" (at 109.22 55.88 0)
-      (effects (font (size 1.27 1.27)) (justify bottom) hide)
-    )
-    (property "DESCRIPTION" "White LED Indication - Discrete 3.3V 2-SMD, No Lead" (at 109.22 55.88 0)
-      (effects (font (size 1.27 1.27)) (justify bottom) hide)
-    )
-    (property "PACKAGE" "SMD-2 Inolux" (at 109.22 55.88 0)
-      (effects (font (size 1.27 1.27)) (justify bottom) hide)
-    )
-    (property "PRICE" "None" (at 109.22 55.88 0)
-      (effects (font (size 1.27 1.27)) (justify bottom) hide)
-    )
-    (property "Package" "SMD-2 Inolux" (at 109.22 55.88 0)
-      (effects (font (size 1.27 1.27)) (justify bottom) hide)
-    )
-    (property "Check_prices" "https://www.snapeda.com/parts/IN-S124ARUW/Inolux/view-part/?ref=eda" (at 109.22 55.88 0)
-      (effects (font (size 1.27 1.27)) (justify bottom) hide)
-    )
-    (property "Price" "None" (at 109.22 55.88 0)
-      (effects (font (size 1.27 1.27)) (justify bottom) hide)
-    )
-    (property "SnapEDA_Link" "https://www.snapeda.com/parts/IN-S124ARUW/Inolux/view-part/?ref=snap" (at 109.22 55.88 0)
-      (effects (font (size 1.27 1.27)) (justify bottom) hide)
-    )
-    (property "MP" "IN-S124ARUW" (at 109.22 55.88 0)
-      (effects (font (size 1.27 1.27)) (justify bottom) hide)
-    )
-    (property "DIGIKEY-PURCHASE-URL" "https://snapeda.com/shop?store=DigiKey&id=2130298" (at 109.22 55.88 0)
-      (effects (font (size 1.27 1.27)) (justify bottom) hide)
-    )
-    (property "Description" "\nWhite - LED Indication - Discrete 3.3V 2-SMD, No Lead\n" (at 109.22 55.88 0)
-      (effects (font (size 1.27 1.27)) (justify bottom) hide)
-    )
-    (property "Availability" "In Stock" (at 109.22 55.88 0)
-      (effects (font (size 1.27 1.27)) (justify bottom) hide)
-    )
-    (property "AVAILABILITY" "Warning" (at 109.22 55.88 0)
-      (effects (font (size 1.27 1.27)) (justify bottom) hide)
-    )
-    (property "MAXIMUM_PACKAGE_HEIGHT" "0.3mm" (at 109.22 55.88 0)
-      (effects (font (size 1.27 1.27)) (justify bottom) hide)
-    )
-    (pin "A")
-    (pin "C")
-    (instances
-      (project "nightLight"
-        (path "/203033dd-6a13-4262-9a98-8b29445e90e8"
-          (reference "D1") (unit 1)
-        )
-      )

Commit message: Finished new design, needs to be reviewed and rid of errors
Parts:
- removed C3: 22uF, Capacitor_SMD:C_1206_3216Metric, symbol Device:C
- removed R1: 0, Resistor_SMD:R_1206_3216Metric, symbol Device:R_US
- removed U1: MCP73831-2-OT, Package_TO_SOT_SMD:SOT-23-5, symbol Battery_Management:MCP73831-2-OT
- added FID1: Fiducial, Fiducial:Fiducial_1.5mm_Mask3mm, symbol Mechanical:Fiducial
- added IC2: MCP73123T-22SI_MF, MCP73123T-22SI_MF:SON50P300X300X100-11N-D, symbol MCP73123T-22SI_MF:MCP73123T-22SI_MF
- added U3, U4, U5, U6, U7, U8, U9: ~, myFootprintDesigns:fireflyTouchNB, symbol myDesigns:Firefly_Symbol
- C1, C2, C5, C6, C7: footprint Capacitor_SMD:C_1206_3216Metric -> Capacitor_SMD:C_0805_2012Metric
- C4: value 10uF -> 4.7uF; footprint Capacitor_SMD:C_1206_3216Metric -> Capacitor_SMD:C_0805_2012Metric
- J5: footprint Connector_PinHeader_2.54mm:PinHeader_1x03_P2.54mm_Vertical_SMD_Pin1Left -> myFootprintDesigns:spares_1*3
- LED1: footprint INS124ARUW -> KiCad-SMTLED:INS124ARUW
- R10, R11, R12, R13, R2, R3, R4, R6, R7, R8, R9: footprint Resistor_SMD:R_1206_3216Metric -> Resistor_SMD:R_0805_2012Metric
- R5: value 10k -> 5.1K; footprint Resistor_SMD:R_1206_3216Metric -> Resistor_SMD:R_0805_2012Metric
Connections:
- net vBATT is gone; now on net VBATT: C1.1, IC1.3 (VIN), L1.1, R3.1, R9.1
- net GND: now also IC2.11 (EP), IC2.8 (VSS_1), IC2.9 (VSS_2)
- net VBATT: now also IC2.3 (VBAT_1), IC2.4 (VBAT_2)
- net at C2.1, J1.A9 (VBUS), J1.B9 (VBUS): now also LED1.2 (A), IC2.1 (VDD_1), IC2.2 (VDD_2); no longer R6.1
- net at LED1.1 (K): now also R6.1
- net at R6.2: now also IC2.7 (STAT); no longer LED1.2 (A)
- net at R5.1: now also IC2.10 (PROG)
- no-connect marks 2 -> 4
Other:
- moved on the sheet: BT1, C4, C5, LED1, R6

Commit message: generated fab files
Parts:
- R10, R9: value 100k -> 0
Changed lines of the file:
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@@
       (effects (font (size 1.27 1.27)) (justify left))
     )
-    (property "Value" "100k" (at 196.85 132.08 0)
+    (property "Value" "0" (at 196.85 132.08 0)
       (effects (font (size 1.27 1.27)) (justify left))
     )
@@
       (effects (font (size 1.27 1.27)) (justify left))
     )
-    (property "Value" "100k" (at 196.85 144.78 0)
+    (property "Value" "0" (at 196.85 144.78 0)
       (effects (font (size 1.27 1.27)) (justify left))
     )

Commit message: messing around during testing
Parts:
- added U1: MCP809T-270I_TT, MCP809T-270I_TT:SOT95P237X112-3N, symbol MCP809T-270I_TT:MCP809T-270I_TT
- R3: value 750K -> 100K
Connections:
- net GND: now also U1.1 (VSS)
- net VBATT: now also U1.3 (VDD); no longer R3.1
- new net ~{RST}: R3.1, U1.2 (~{RST})
Other:
- moved on the sheet: B1, C1, C5, C6, C7, IC1, J2, J3, J4, J5, J6, L1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
