File: hardware/board-files/nightLight-r3/chargeController.kicad_sch (KiCad schematic)
At the start: 10 parts, among them IC3 MCP73123T-22SI_MF, J7 USB_C_Receptacle_PowerOnly_6P

Commit message: first layout revision
Parts:
- renumbered BT2 to BT1, C5 to C4, C8 to C5, IC3 to IC2, J7 to J1, LED2 to LED1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
