File: hardware/board-files/nightLight-r3/MCU.kicad_sch (KiCad schematic)
At the start: 14 parts, among them J1 Conn_01x03, J2 Conn_01x03, J3 Conn_01x03, J4 Conn_01x03, J5 Conn_01x05_Pin, SW1 TILT, U1 ATtiny1614-SS

Commit message: first layout revision
Parts:
- R12: renamed from R6; value 0 -> 1M
- R14: renamed from R9; value 0 -> 1M
- renumbered C4 to C6, C6 to C7, J5 to J2, J4 to J3, J1 to J4, J2 to J5, J3 to J6, R10 to R13, U1 to U8
Connections:
- net FET_CONTROL: now also U8.5 (PA7); no longer U8.9 (PB0)
- net TILT_SW: now also U8.9 (PB0); no longer U8.5 (PA7)

Commit message: rev3 done, errors eliminated
Parts:
- added R15, R16: 0, Resistor_SMD:R_0805_2012Metric, symbol Device:R_US
- J4, J5, J6: footprint Connector_PinHeader_2.54mm:PinHeader_1x03_P2.54mm_Vertical_SMD_Pin1Left -> myFootprintDesigns:fairy_conn
Connections:
- net RX: now also R15.1; no longer J2.3 (Pin_3)
- net TX: now also R16.1; no longer J2.2 (Pin_2)
- new net: J2.2 (Pin_2), R16.2
- new net: J2.3 (Pin_3), R15.2
Changed lines of the file:
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@@
+    (stroke (width 0) (type default))
+  )
+  (wire (pts (xy 189.23 63.5) (xy 190.5 63.5))
     (stroke (width 0) (type default))
   )
@@
     (stroke (width 0) (type default))
   )
+  (wire (pts (xy 180.34 63.5) (xy 181.61 63.5))
+    (stroke (width 0) (type default))
+  )
   (wire (pts (xy 115.57 63.5) (xy 124.46 63.5))
     (stroke (width 0) (type default))
@@
     (stroke (width 0) (type default))
   )
-  (wire (pts (xy 185.42 63.5) (xy 190.5 63.5))
-    (stroke (width 0) (type default))
-  )
   (wire (pts (xy 139.7 52.07) (xy 139.7 55.88))
     (stroke (width 0) (type default))
@@
     (stroke (width 0) (type default))
   )
+  (wire (pts (xy 189.23 66.04) (xy 190.5 66.04))
+    (stroke (width 0) (type default))
+  )
   (wire (pts (xy 154.94 78.74) (xy 158.75 78.74))
     (stroke (width 0) (type default))
@@
     (stroke (width 0) (type default))
   )
+  (wire (pts (xy 180.34 66.04) (xy 181.61 66.04))
+    (stroke (width 0) (type default))
+  )
   (wire (pts (xy 154.94 76.2) (xy 158.75 76.2))
     (stroke (width 0) (type default))
@@
     (stroke (width 0) (type default))
   )
-  (wire (pts (xy 185.42 66.04) (xy 190.5 66.04))
-    (stroke (width 0) (type default))
-  )
   (wire (pts (xy 99.06 91.44) (xy 99.06 90.805))
     (stroke (width 0) (type default))
@@
     (stroke (width 0) (type default))
   )
-  (wire (pts (xy 185.42 60.96) (xy 190.5 60.96))
+  (wire (pts (xy 184.15 60.96) (xy 190.5 60.96))
     (stroke (width 0) (type default))
   )
@@
     (effects (font (size 1.27 1.27)) (justify right bottom))
   )
-  (label "RX" (at 185.42 63.5 180) (fields_autoplaced)
+  (label "RX" (at 180.34 63.5 180) (fields_autoplaced)
     (effects (font (size 1.27 1.27)) (justify right bottom))
   )
@@
     (effects (font (size 1.27 1.27)) (justify left bottom))
   )
-  (label "UPDI" (at 185.42 60.96 180) (fields_autoplaced)
+  (label "UPDI" (at 184.15 60.96 180) (fields_autoplaced)
     (effects (font (size 1.27 1.27)) (justify right bottom))
   )
@@
     (effects (font (size 1.27 1.27)) (justify right bottom))
   )
-  (label "TX" (at 185.42 66.04 180) (fields_autoplaced)
+  (label "TX" (at 180.34 66.04 180) (fields_autoplaced)
     (effects (font (size 1.27 1.27)) (justify right bottom))
   )
@@
     )
   )
+  (symbol (lib_id "Device:R_US") (at 185.42 63.5 90) (unit 1)
+    (in_bom yes) (on_board yes) (dnp no)
+    (property "Reference" "R15" (at 182.88 64.77 90)
+      (effects (font (size 1.27 1.27)))
+    )
+    (property "Value" "0" (at 189.23 62.23 90)
+      (effects (font (size 1.27 1.27)))
+    )
+    (property "Footprint" "Resistor_SMD:R_0805_2012Metric" (at 185.674 62.484 90)
+      (effects (font (size 1.27 1.27)) hide)
+    )
+    (property "Datasheet" "~" (at 185.42 63.5 0)
+      (effects (font (size 1.27 1.27)) hide)
+    )
+    (pin "1")
+    (pin "2")
+    (instances
+      (project "nightLight"
+        (path "/203033dd-6a13-4262-9a98-8b29445e90e8/60503468-aee4-4d11-84bc-8967446d1603"
+          (reference "R15") (unit 1)
+        )
+      )
+    )
+  )
   (symbol (lib_id "power:GND") (at 99.06 95.25 0) (unit 1)
     (in_bom yes) (on_board yes) (dnp no) (fields_autoplaced)
@@
       (effects (font (size 1.27 1.27)) (justify left) hide)
     )
-    (property "Footprint" "Connector_PinHeader_2.54mm:PinHeader_1x03_P2.54mm_Vertical_SMD_Pin1Left" (at 104.14 90.805 0)
+    (property "Footprint" "myFootprintDesigns:fairy_conn" (at 104.14 90.805 0)
       (effects (font (size 1.27 1.27)) hide)
     )
@@
       (effects (font (size 1.27 1.27)) (justify left) hide)
     )
-    (property "Footprint" "Connector_PinHeader_2.54mm:PinHeader_1x03_P2.54mm_Vertical_SMD_Pin1Left" (at 104.14 112.395 0)
+    (property "Footprint" "myFootprintDesigns:fairy_conn" (at 104.14 112.395 0)
       (effects (font (size 1.27 1.27)) hide)
     )
@@
         (path "/203033dd-6a13-4262-9a98-8b29445e90e8/60503468-aee4-4d11-84bc-8967446d1603"
           (reference "#PWR019") (unit 1)
+        )
+      )
+    )
+  )
+  (symbol (lib_id "Device:R_US") (at 185.42 66.04 90) (unit 1)
+    (in_bom yes) (on_board yes) (dnp no)
+    (property "Reference" "R16" (at 182.88 62.23 90)
+      (effects (font (size 1.27 1.27)))
+    )
+    (property "Value" "0" (at 189.23 64.77 90)
+      (effects (font (size 1.27 1.27)))
+    )
+    (property "Footprint" "Resistor_SMD:R_0805_2012Metric" (at 185.674 65.024 90)
+      (effects (font (size 1.27 1.27)) hide)
+    )
+    (property "Datasheet" "~" (at 185.42 66.04 0)
+      (effects (font (size 1.27 1.27)) hide)
+    )
+    (pin "1")
+    (pin "2")
+    (instances
+      (project "nightLight"
+        (path "/203033dd-6a13-4262-9a98-8b29445e90e8/60503468-aee4-4d11-84bc-8967446d1603"
+          (reference "R16") (unit 1)
         )
       )
@@
       (effects (font (size 1.27 1.27)) (justify left) hide)
     )
-    (property "Footprint" "Connector_PinHeader_2.54mm:PinHeader_1x03_P2.54mm_Vertical_SMD_Pin1Left" (at 104.14 133.35 0)
-      (effects (font (size 1.27 1.27)) hide)
-    )
+    (property "Footprint" "myFootprintDesigns:fairy_conn" (at 104.14 133.35 0)
+      (effects (font (size 1.27 1.27)) hide)
+    )
