File: hardware/board-files/nightLight-r3/vReg.kicad_sch (KiCad schematic)
At the start: 14 parts, among them IC1 PAM2401SCADJ, Q1 AO3400A, Q2 AO3401A

Commit message: PCB R3 Finished and ordered
Parts:
- added Q3: AO3401A, Package_TO_SOT_SMD:SOT-23, symbol Transistor_FET:AO3401A
Connections:
- net GND: now also Q3.1 (G)
- net Vbatt: now also Q3.3 (D); no longer Q2.3 (D), R2.1
- new net: Q2.3 (D), Q3.2 (S), R2.1
Other:
- note added: "Reverse polarity protection"
Changed lines of the file:
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@@
   (junction (at 115.57 71.12) (diameter 0) (color 0 0 0 0)
   )
+  (junction (at 146.05 66.04) (diameter 0) (color 0 0 0 0)
+  )
   (junction (at 97.79 71.12) (diameter 0) (color 0 0 0 0)
   )
   (junction (at 208.28 113.03) (diameter 0) (color 0 0 0 0)
-  )
-  (junction (at 146.05 66.04) (diameter 0) (color 0 0 0 0)
   )
   (junction (at 137.16 78.74) (diameter 0) (color 0 0 0 0)
@@
     (stroke (width 0) (type default))
   )
+  (wire (pts (xy 146.05 44.45) (xy 146.05 52.07))
+    (stroke (width 0) (type default))
+  )
   (wire (pts (xy 224.79 111.76) (xy 224.79 113.03))
     (stroke (width 0) (type default))
@@
     (stroke (width 0) (type default))
   )
+  (wire (pts (xy 146.05 62.23) (xy 146.05 66.04))
+    (stroke (width 0) (type default))
+  )
   (wire (pts (xy 146.05 128.27) (xy 146.05 127))
     (stroke (width 0) (type default))
@@
     (stroke (width 0) (type default))
   )
-  (wire (pts (xy 146.05 57.15) (xy 146.05 66.04))
+  (wire (pts (xy 157.48 57.15) (xy 157.48 60.96))
     (stroke (width 0) (type default))
   )
@@
     (stroke (width 0) (type default))
   )
+  (wire (pts (xy 153.67 57.15) (xy 157.48 57.15))
+    (stroke (width 0) (type default))
+  )
   (wire (pts (xy 168.91 129.54) (xy 168.91 139.7))
     (stroke (width 0) (type default))
@@
   (wire (pts (xy 151.13 110.49) (xy 151.13 119.38))
     (stroke (width 0) (type default))
+  )
+  (text "Reverse polarity protection" (at 151.13 53.34 0)
+    (effects (font (size 2 2) (color 237 0 0 1)) (justify left bottom))
   )
   (text "LVD Circuit\n" (at 101.6 58.42 0)
@@
     (effects (font (size 1.27 1.27)) (justify right))
   )
-  (hierarchical_label "Vbatt" (shape input) (at 146.05 57.15 90) (fields_autoplaced)
+  (hierarchical_label "Vbatt" (shape input) (at 146.05 44.45 90) (fields_autoplaced)
     (effects (font (size 1.27 1.27)) (justify left))
   )
@@
     )
   )
+  (symbol (lib_id "Transistor_FET:AO3401A") (at 148.59 57.15 0) (mirror y) (unit 1)
+    (in_bom yes) (on_board yes) (dnp no)
+    (property "Reference" "Q3" (at 142.24 55.88 0)
+      (effects (font (size 1.27 1.27)) (justify left))
+    )
+    (property "Value" "AO3401A" (at 142.24 58.42 0)
+      (effects (font (size 1.27 1.27)) (justify left))
+    )
+    (property "Footprint" "Package_TO_SOT_SMD:SOT-23" (at 143.51 59.055 0)
+      (effects (font (size 1.27 1.27) italic) (justify left) hide)
+    )
+    (property "Datasheet" "http://www.aosmd.com/pdfs/datasheet/AO3401A.pdf" (at 143.51 60.96 0)
+      (effects (font (size 1.27 1.27)) (justify left) hide)
+    )
+    (pin "3")
+    (pin "2")
+    (pin "1")
+    (instances
+      (project "nightLight"
+        (path "/203033dd-6a13-4262-9a98-8b29445e90e8/e6a767d4-c228-4ec6-8577-23f8c70359e3"
+          (reference "Q3") (unit 1)
+        )
+      )
+    )
+  )
   (symbol (lib_id "power:GND") (at 146.05 139.7 0) (unit 1)
     (in_bom yes) (on_board yes) (dnp no) (fields_autoplaced)
@@
         )
       )
+    )
+  )
+  (symbol (lib_id "power:GND") (at 157.48 60.96 0) (unit 1)
+    (in_bom yes) (on_board yes) (dnp no) (fields_autoplaced)
+    (property "Reference" "#PWR032" (at 157.48 67.31 0)
+      (effects (font (size 1.27 1.27)) hide)
+    )
+    (property "Value" "GND" (at 157.48 66.04 0)
+      (effects (font (size 1.27 1.27)))
+    )
+    (property "Footprint" "" (at 157.48 60.96 0)
+      (effects (font (size 1.27 1.27)) hide)
+    )
+    (property "Datasheet" "" (at 157.48 60.96 0)
+      (effects (font (size 1.27 1.27)) hide)
+    )
+    (pin "1")
+    (instances
+      (project "nightLight"
+        (path "/203033dd-6a13-4262-9a98-8b29445e90e8/e6a767d4-c228-4ec6-8577-23f8c70359e3"
+          (reference "#PWR032") (unit 1)
+        )
+      )
